File: Issue1.kicad_pcb (KiCad board)
At the start: 2 copper layers, 160 x 35.6 mm, 27 parts, among them IC1 74LS157, IC10 4532, IC11 74LS32, IC12 74LS00, IC2 74LS157, IC3 4532, IC4 4532, IC5 4532, IC6 4532, IC7 4532, IC8 4532, IC9 4532

Commit message: Correct  C9 & C10 Values
Correct  C9 & C10 Values
Parts:
- C10: value 100pF -> 47pF
- C9: value 47pF -> 100pF
